File: BufferCorrente/BufferCorrente.kicad_sch (KiCad schematic)
At the start: 38 parts, among them J1 INPUT, J2 OUTPUT, Q1 BD138, Q2 BD138, Q3 BD138, U1 LM318N

Commit message: Aggiornata la PCB del buffer in corrente con coponenti SMD e groud plane
Parts:
- removed C13, C17: 22uF, Capacitor_THT:C_Rect_L7.0mm_W2.0mm_P5.00mm, symbol Device:C
- removed C3, C4: 12pF, Capacitor_THT:C_Rect_L7.0mm_W2.0mm_P5.00mm, symbol Device:C
- removed R3: 10K, Resistor_THT:R_Axial_DIN0207_L6.3mm_D2.5mm_P7.62mm_Horizontal, symbol Device:R
- removed U1: LM318N, Package_DIP:CERDIP-8_W7.62mm_SideBrazed_Socket, symbol Amplifier_Operational:LM318N
- added C13, C17: 22uF, Capacitor_Tantalum_SMD:CP_EIA-3216-18_Kemet-A, symbol Device:C_Polarized
- added H1, H2, H3, H4: MountingHole_Pad, MountingHole:MountingHole_3.2mm_M3_Pad_Via, symbol Mechanical:MountingHole_Pad
- added J3: Differenzial, TerminalBlock:TerminalBlock_Xinya_XY308-2.54-3P_1x03_P2.54mm_Horizontal, symbol Connector:Screw_Terminal_01x03
- added U1: OPA134, Package_DIP:DIP-8_W7.62mm_Socket, symbol Amplifier_Operational:OPA134
- C1, C2: value 100nF -> 10nF; footprint Capacitor_THT:C_Rect_L7.0mm_W2.0mm_P5.00mm -> Capacitor_SMD:C_0402_1005Metric
- C10, C15: footprint Capacitor_THT:C_Rect_L7.0mm_W2.0mm_P5.00mm -> Capacitor_SMD:C_1206_3216Metric
- C11, C12, C14, C16, C9: footprint Capacitor_THT:C_Rect_L7.0mm_W2.0mm_P5.00mm -> Capacitor_SMD:C_0402_1005Metric
- D1, D2, D5: footprint Diode_THT:D_DO-35_SOD27_P7.62mm_Horizontal -> Diode_SMD:D_SOD-123
- D6, D7: footprint Diode_THT:D_DO-35_SOD27_P7.62mm_Horizontal -> Diode_SMD:D_SOD-123F
- R1, R2: footprint Resistor_THT:R_Axial_DIN0207_L6.3mm_D2.5mm_P7.62mm_Horizontal -> Resistor_SMD:R_0201_0603Metric
- R10, R11: footprint Resistor_THT:R_Axial_DIN0207_L6.3mm_D2.5mm_P7.62mm_Horizontal -> Resistor_THT:R_Axial_DIN0414_L11.9mm_D4.5mm_P15.24mm_Horizontal
- R4, R5, R6, R7, R8, R9: footprint Resistor_THT:R_Axial_DIN0207_L6.3mm_D2.5mm_P7.62mm_Horizontal -> Resistor_SMD:R_1206_3216Metric
Connections:
- net +16V: now also U1.7 (V+)
- net -16V: now also U1.4 (V-)
- net GND: now also H1.1, H2.1, H3.1, H4.1, J3.1 (Pin_1)
- net at C12.2, C16.1, J2.1 (Pin_1)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: now also C13.2, C17.1, U1.2 (-)
- net at C16.2, R8.2, R9.1: now also C17.2
- net at C12.1, R6.1, R7.2: now also C13.1
- net at D1.2 (A), D2.1 (K), R1.2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: now also U1.3 (+)
- net at Q1.2 (C), Q2.3 (B), R5.2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: now also U1.6
- new net VCC: J3.3 (Pin_3)
- new net VEE: J3.2 (Pin_2)
